Commit message: Added 360 bot algorithm

File: urdf/micromouse_orig.urdf (robot description, URDF)
Before this commit: robot my_mm_robot, 6 links, 5 joints
Links:
- removed link link_back_wheel
- removed link link_front_wheel
- link link_chassis: mass 0 -> 0.5; geometry collision box size=0.07 0.07 0.02; collision sphere radius=0.005
- link link_left_wheel: mass 0 -> 0.2; geometry collision cylinder length=0.01 radius=0.02; visual cylinder length=0.01 radius=0.02
- link link_right_wheel: mass 0 -> 0.2; geometry collision cylinder length=0.01 radius=0.02; visual cylinder length=0.01 radius=0.02
- link sensor_laser: mass 0 -> 0.01
Joints:
- removed joint joint_back_wheel
- removed joint joint_front_wheel
- joint joint_left_wheel: origin xyz=0.04 0 0 rpy=0 0 0 -> xyz=0.04 0.02 0 rpy=0 0 0
- joint joint_right_wheel: origin xyz=-0.04  0    0 rpy=0 0 0 -> xyz=-0.04  0.02    0 rpy=0 0 0
- joint joint_sensor_laser: origin xyz=0    0    0.02 rpy=0  0  -1.57 -> xyz=0    0    0.01 rpy=0  0  -1.57

Commit message: Update micromouse_orig.urdf

File: urdf/micromouse_orig.urdf (robot description, URDF)
Before this commit: robot my_mm_robot, 4 links, 3 joints
Links:
- added link link_back_wheel, mass 0.00001; collision cylinder length=0.01 radius=0.015; visual cylinder length=0.01 radius=0.015
- added link link_front_wheel, mass 0.00001; collision cylinder length=0.01 radius=0.015; visual cylinder length=0.01 radius=0.015
- link link_chassis: mass 0.5 -> 0; geometry collision box size=0.07 0.07 0.02; visual box size=0.07 0.07 0.02
- link link_left_wheel: mass 0.2 -> 0.00001; geometry collision cylinder length=0.01 radius=0.015; visual cylinder length=0.01 radius=0.015
- link link_right_wheel: mass 0.2 -> 0.00001; geometry collision cylinder length=0.01 radius=0.015; visual cylinder length=0.01 radius=0.015
Joints:
- added joint joint_back_wheel: type continuous, parent link_chassis, child link_back_wheel, origin xyz=0  0.04    0 rpy=0 0 0, axis 0 1 0, limit effort=5 velocity=6
- added joint joint_front_wheel: type continuous, parent link_chassis, child link_front_wheel, origin xyz=0  -0.04    0 rpy=0 0 0, axis 0 1 0, limit effort=5 velocity=6
- joint joint_left_wheel: origin xyz=0.04 0.02 0 rpy=0 0 0 -> xyz=0.04 0 0 rpy=0 0 0
- joint joint_right_wheel: origin xyz=-0.04  0.02    0 rpy=0 0 0 -> xyz=-0.04  0    0 rpy=0 0 0
- joint joint_sensor_laser: origin xyz=0    0    0.01 rpy=0  0  -1.57 -> xyz=0    0    0.02 rpy=0  0  -1.57
