Commit message: Update micromouse_robot.urdf

File: urdf/micromouse_robot.urdf (robot description, URDF)
Before this commit: robot my_mm_robot, 6 links, 5 joints
Links:
- link link_back_wheel: geometry collision cylinder length=0.01 radius=0.015; visual cylinder length=0.01 radius=0.015
- link link_chassis: geometry collision box size=0.07 0.07 0.02; visual box size=0.07 0.07 0.02
- link link_front_wheel: geometry collision cylinder length=0.01 radius=0.015; visual cylinder length=0.01 radius=0.015
- link link_left_wheel: geometry collision cylinder length=0.01 radius=0.015; visual cylinder length=0.01 radius=0.015
- link link_right_wheel: geometry collision cylinder length=0.01 radius=0.015; visual cylinder length=0.01 radius=0.015
Joints:
- joint joint_back_wheel: axis 1 0 0 -> 0 1 0; origin xyz=0  0.004    0 rpy=0 0 0 -> xyz=0  0.04    0 rpy=0 0 0
- joint joint_front_wheel: axis 1 0 0 -> 0 1 0; origin xyz=0  -0.004    0 rpy=0 0 0 -> xyz=0  -0.04    0 rpy=0 0 0
- joint joint_left_wheel: origin xyz=0.004 0 0 rpy=0 0 0 -> xyz=0.04 0 0 rpy=0 0 0
- joint joint_right_wheel: origin xyz=-0.004  0    0 rpy=0 0 0 -> xyz=-0.04  0    0 rpy=0 0 0
- joint joint_sensor_laser: origin xyz=0    0    0.01 rpy=0  0  -1.57 -> xyz=0    0    0.02 rpy=0  0  -1.57

Commit message: Update micromouse_robot.urdf

File: urdf/micromouse_robot.urdf (robot description, URDF)
Before this commit: robot my_mm_robot, 6 links, 5 joints
Links:
- link link_back_wheel: mass 0.2 -> 0.00001
- link link_chassis: mass 0.5 -> 0
- link link_front_wheel: mass 0.2 -> 0.00001
- link link_left_wheel: mass 0.2 -> 0.00001
- link link_right_wheel: mass 0.2 -> 0.00001

Commit message: Changed regions and added sensor exchange function

File: urdf/micromouse_robot.urdf (robot description, URDF)
Before this commit: robot my_mm_robot, 6 links, 5 joints
Links:
- link link_back_wheel: mass 0 -> 0.2
- link link_chassis: mass 0 -> 0.5
- link link_front_wheel: mass 0 -> 0.2
- link link_left_wheel: mass 0 -> 0.2
- link link_right_wheel: mass 0 -> 0.2
- link sensor_laser: mass 0 -> 0.01
